File: electronics/digital/digital.sch (KiCad schematic (older format))
At the start: 50 parts

Commit message: add headers and usb ports
Parts:
- added C? (x2): 100n, symbol C
- added J? (x2): USB_A, symbol USB_A
- added P? (x2): USB_CABLE, symbol CONN_01X03
- added P?: EXTERNAL_HEADER, symbol CONN_01X10
- added P?: INTERNAL_HEADER, symbol CONN_01X10
- added P?: CONN_02X05, symbol CONN_02X05
Connections:
- wire segments 126 -> 198
Other:
- moved on the sheet: J?, P?

Commit message: ran annotation
Parts:
- gave numbers to parts that had none: 59

Commit message: fix ERC errors
Connections:
- wire segments 198 -> 170
- no-connect marks 0 -> 1

Commit message: sync to pcb
Parts:
- removed P6: EXTERNAL_HEADER, symbol CONN_01X10
- removed P8: INTERNAL_HEADER, symbol CONN_01X10
- removed Q1, Q2, Q5: MOSFET_P, symbol MOSFET_P
- added P6: EXTERNAL_HEADER, Pin_Headers:Pin_Header_Straight_2x05, symbol CONN_02X05
- added P8: INTERNAL_HEADER, Pin_Headers:Pin_Header_Straight_2x05, symbol CONN_02X05
- added Q1, Q2, Q5: MOS_P_123, Transistors_SMD:sot23, symbol MOS_P_123
- BT1: footprint (none) -> BAT-CR2032:BAT-CR2032
- C1, C3: footprint (none) -> Capacitors_ThroughHole:Capacitor16x25RM7.5
- C2, C4, C5, C6, C7, C8: footprint (none) -> Capacitors_ThroughHole:Capacitor6MMDiscRM5
- D1, D2, P10, P2, P9: footprint (none) -> Pin_Headers:Pin_Header_Straight_1x02
- J1, J2: footprint (none) -> usb:USB_A
- J3: footprint (none) -> Connect:RJ45_8
- L1: footprint (none) -> SMD_Packages:SMD-1206
- P1: footprint (none) -> barrel:BARREL_JACK
- P11: footprint (none) -> Pin_Headers:Pin_Header_Straight_1x05
- P3, P4: footprint (none) -> Pin_Headers:Pin_Header_Straight_1x03
- P5: footprint (none) -> Pin_Headers:Pin_Header_Straight_1x10
- P7: value CONN_02X05 -> POWER_OUT; footprint (none) -> Pin_Headers:Pin_Header_Straight_2x05
- Q10, Q3, Q4, Q6, Q7, Q9: footprint (none) -> Discret:TO92-123
- Q8: footprint (none) -> Transistors_TO-220:TO-220_FET-GDS_Vertical
- R1, R10, R11, R12, R13, R14, R15, R16, R17, R18, R19, R2, R20, R21, R3, R4, R5, R6, R7, R8, R9: footprint (none) -> Resistors_ThroughHole:Resistor_Horizontal_RM10mm
- U1: footprint (none) -> Power_Integrations:SO-8
- X1: footprint (none) -> QMONTRE_P:QMONTRE_P
Connections:
- wire segments 170 -> 190

Commit message: add rj45
Parts:
- removed P5: NETWORK, Pin_Headers:Pin_Header_Straight_1x10, symbol CONN_01X10
- added P5: NETWORK_CABLE, rj45:RJ45_SOLDER, symbol CONN_01X08
- J3: footprint Connect:RJ45_8 -> rj45:RJ45_8_BIG
- P6: footprint Pin_Headers:Pin_Header_Straight_2x05 -> Pin_Headers:Pin_Header_Angled_2x05
Connections:
- wire segments 190 -> 185

Commit message: add fuse
Parts:
- added F?: FUSE, symbol FUSE
Connections:
- wire segments 185 -> 186
Other:
- moved on the sheet: P1
Changed lines of the file:
@@
 L CONN_01X02 P1
 U 1 1 550C91AB
-P 1500 1150
-F 0 "P1" H 1500 1300 50  0000 C CNN
-F 1 "POWER_IN" H 1500 1000 50  0000 C CNN
-F 2 "barrel:BARREL_JACK" H 1500 1150 60  0001 C CNN
-F 3 "" H 1500 1150 60  0000 C CNN
-	1    1500 1150
+P 1100 1150
+F 0 "P1" H 1100 1300 50  0000 C CNN
+F 1 "POWER_IN" H 1100 1000 50  0000 C CNN
+F 2 "barrel:BARREL_JACK" H 1100 1150 60  0001 C CNN
+F 3 "" H 1100 1150 60  0000 C CNN
+	1    1100 1150
 	-1   0    0    -1
 $EndComp
@@
 L GND #PWR09
 U 1 1 550CD265
-P 1800 1650
-F 0 "#PWR09" H 1800 1400 60  0001 C CNN
-F 1 "GND" H 1800 1500 60  0001 C CNN
-F 2 "" H 1800 1650 60  0000 C CNN
-F 3 "" H 1800 1650 60  0000 C CNN
-	1    1800 1650
+P 1400 1650
+F 0 "#PWR09" H 1400 1400 60  0001 C CNN
+F 1 "GND" H 1400 1500 60  0001 C CNN
+F 2 "" H 1400 1650 60  0000 C CNN
+F 3 "" H 1400 1650 60  0000 C CNN
+	1    1400 1650
 	1    0    0    -1
 $EndComp
@@
 	4400 4900 4500 4900
 Wire Wire Line
-	1700 1100 2450 1100
+	1950 1100 2450 1100
 Wire Wire Line
 	2100 950  2100 1200
@@
 AMP_SEL
 Wire Wire Line
-	1800 1200 1800 1650
-Wire Wire Line
-	1800 1200 1700 1200
+	1400 1200 1400 1650
+Wire Wire Line
+	1400 1200 1300 1200
 $Comp
 L +5V #PWR020
@@
 L PWR_FLAG #FLG048
 U 1 1 5510E698
-P 1600 1600
-F 0 "#FLG048" H 1600 1695 30  0001 C CNN
-F 1 "PWR_FLAG" H 1600 1780 30  0001 C CNN
-F 2 "" H 1600 1600 60  0000 C CNN
-F 3 "" H 1600 1600 60  0000 C CNN
-	1    1600 1600
+P 1200 1600
+F 0 "#FLG048" H 1200 1695 30  0001 C CNN
+F 1 "PWR_FLAG" H 1200 1780 30  0001 C CNN
+F 2 "" H 1200 1600 60  0000 C CNN
+F 3 "" H 1200 1600 60  0000 C CNN
+	1    1200 1600
 	-1   0    0    1
 $EndComp
 Wire Wire Line
-	1600 1600 1600 1500
-Wire Wire Line
-	1600 1500 1800 1500
-Connection ~ 1800 1500
+	1200 1600 1200 1500
+Wire Wire Line
+	1200 1500 1400 1500
+Connection ~ 1400 1500
 $Comp
 L PWR_FLAG #FLG049
@@
 	0    1    1    0
 $EndComp
+$Comp
+L FUSE F?
+U 1 1 55292D4A
+P 1700 1100
+F 0 "F?" H 1800 1150 40  0000 C CNN
+F 1 "FUSE" H 1600 1050 40  0000 C CNN
+F 2 "" H 1700 1100 60  0000 C CNN
+F 3 "" H 1700 1100 60  0000 C CNN
+	1    1700 1100
+	1    0    0    -1
+$EndComp
+Wire Wire Line
+	1450 1100 1300 1100
 $EndSCHEMATC

Commit message: arrange transistors
Parts:
- removed R12, R13: 10, Resistors_ThroughHole:Resistor_Horizontal_RM10mm, symbol R
- F1: renamed from F?; footprint (none) -> Capacitors_ThroughHole:Capacitor6MMDiscRM5
- Q8: footprint Transistors_TO-220:TO-220_FET-GDS_Vertical -> SMD_Packages:DPAK-2-1EP_GDS
Connections:
- wire segments 186 -> 218
Other:
- moved on the sheet: D1, D2, R1, R2
Changed lines of the file:
@@
-$EndComp
-$Comp
-L R R12
-U 1 1 550C91CE
-P 6150 5000
-F 0 "R12" H 6250 5050 40  0000 C CNN
-F 1 "10" H 6250 4950 40  0000 C CNN
-F 2 "Resistors_ThroughHole:Resistor_Horizontal_RM10mm" V 6080 5000 30  0001 C CNN
-F 3 "" H 6150 5000 30  0000 C CNN
-	1    6150 5000
-	1    0    0    -1
 $EndComp
 $Comp
@@
 F 0 "Q8" H 6050 6400 60  0000 R CNN
 F 1 "MOSFET_N" H 6210 6050 60  0001 R CNN
-F 2 "Transistors_TO-220:TO-220_FET-GDS_Vertical" H 6200 6200 60  0001 C CNN
+F 2 "SMD_Packages:DPAK-2-1EP_GDS" H 6200 6200 60  0001 C CNN
 F 3 "" H 6200 6200 60  0000 C CNN
 	1    6200 6200
@@
 L LED D1
 U 1 1 550C91CD
-P 6150 4450
-F 0 "D1" V 6000 4500 50  0000 C CNN
-F 1 "LED" H 6150 4350 50  0000 C CNN
-F 2 "Pin_Headers:Pin_Header_Straight_1x02" H 6150 4450 60  0001 C CNN
-F 3 "" H 6150 4450 60  0000 C CNN
-	1    6150 4450
+P 6150 4300
+F 0 "D1" V 6000 4350 50  0000 C CNN
+F 1 "LED" H 6150 4200 50  0000 C CNN
+F 2 "Pin_Headers:Pin_Header_Straight_1x02" H 6150 4300 60  0001 C CNN
+F 3 "" H 6150 4300 60  0000 C CNN
+	1    6150 4300
 	0    1    1    0
 $EndComp
@@
 L R R1
 U 1 1 550DEE92
-P 3050 2550
-F 0 "R1" V 2950 2450 40  0000 C CNN
-F 1 "1" V 3057 2551 40  0000 C CNN
-F 2 "Resistors_ThroughHole:Resistor_Horizontal_RM10mm" V 2980 2550 30  0001 C CNN
-F 3 "" H 3050 2550 30  0000 C CNN
-	1    3050 2550
-	0    1    1    0
+P 6450 4900
+F 0 "R1" H 6350 5100 40  0000 C CNN
+F 1 "1" H 6450 4900 40  0000 C CNN
+F 2 "Resistors_ThroughHole:Resistor_Horizontal_RM10mm" V 6380 4900 30  0001 C CNN
+F 3 "" H 6450 4900 30  0000 C CNN
+	1    6450 4900
+	-1   0    0    -1
 $EndComp
 $Comp
@@
 L R R2
 U 1 1 550DF363
-P 4800 2750
-F 0 "R2" V 4700 2650 40  0000 C CNN
-F 1 "1" V 4807 2751 40  0000 C CNN
-F 2 "Resistors_ThroughHole:Resistor_Horizontal_RM10mm" V 4730 2750 30  0001 C CNN
-F 3 "" H 4800 2750 30  0000 C CNN
-	1    4800 2750
-	0    1    1    0
+P 6150 4900
+F 0 "R2" H 6250 4700 40  0000 C CNN
+F 1 "1" H 6150 4900 40  0000 C CNN
+F 2 "Resistors_ThroughHole:Resistor_Horizontal_RM10mm" V 6080 4900 30  0001 C CNN
+F 3 "" H 6150 4900 30  0000 C CNN
+	1    6150 4900
+	-1   0    0    1
 $EndComp
 $Comp
@@
 	3250 6300 3250 6250
 Wire Wire Line
-	3100 5650 3400 5650
+	3100 5650 3250 5650
+Wire Wire Line
+	3250 5650 3400 5650
 Wire Wire Line
 	3250 5750 3250 5650
@@
 	3700 5950 3700 5850
 Wire Wire Line
-	3700 5100 3700 5450
+	3700 5100 3700 5400
+Wire Wire Line
+	3700 5400 3700 5450
 Wire Wire Line
 	3300 5350 3300 5400
@@
 	4400 4900 4500 4900
 Wire Wire Line
-	1950 1100 2450 1100
-Wire Wire Line
-	2100 950  2100 1200
+	1950 1100 2100 1100
+Wire Wire Line
+	2100 1100 2350 1100
+Wire Wire Line
+	2350 1100 2450 1100
+Wire Wire Line
+	2100 950  2100 1100
+Wire Wire Line
+	2100 1100 2100 1200
 Connection ~ 2100 1100
 Wire Wire Line
-	2350 1000 2350 1200
+	2350 1000 2350 1100
+Wire Wire Line
+	2350 1100 2350 1200
 Connection ~ 2350 1100
 Wire Wire Line
-	3150 4800 3500 4800
+	3150 4800 3300 4800
+Wire Wire Line
+	3300 4800 3500 4800
 Wire Wire Line
 	3300 4850 3300 4800
@@
 	3800 7200 3800 7150
 Wire Wire Line
-	3650 6550 3950 6550
+	3650 6550 3800 6550
+Wire Wire Line
+	3800 6550 3950 6550
 Wire Wire Line
 	3800 6650 3800 6550
@@
 	4250 6850 4250 6750
 Wire Wire Line
-	4250 6050 4250 6350
+	4250 6050 4250 6200
+Wire Wire Line
+	4250 6200 4250 6350
 Wire Wire Line
 	4350 6200 4250 6200
@@
 	5000 5800 4950 5800
 Wire Wire Line
-	4950 5800 4950 6600
+	4950 5800 4950 6200
+Wire Wire Line
+	4950 6200 4950 6600
 Wire Wire Line
 	4950 6600 5000 6600
@@
 Connection ~ 4950 6200
 Wire Wire Line
-	5300 6000 5300 6400
+	5300 6000 5300 6200
+Wire Wire Line
+	5300 6200 5300 6400
 Wire Wire Line
 	5400 6200 5300 6200
@@
 	2100 4050 2100 4000
 Wire Wire Line
-	1950 3400 2250 3400
+	1950 3400 2100 3400
+Wire Wire Line
+	2100 3400 2250 3400
 Wire Wire Line
 	2100 3500 2100 3400
@@
 	2550 3700 2550 3600
 Wire Wire Line
-	2550 2850 2550 3200
+	2550 2850 2550 3150
+Wire Wire Line
+	2550 3150 2550 3200
 Wire Wire Line
 	2150 3100 2150 3150
@@
 Connection ~ 2550 3150
 Wire Wire Line
-	2800 2550 2750 2550
-Wire Wire Line
 	3850 4250 3850 4200
 Wire Wire Line
-	3700 3600 4000 3600
+	3700 3600 3850 3600
+Wire Wire Line
+	3850 3600 4000 3600
 Wire Wire Line
 	3850 3700 3850 3600
@@
 	4300 3900 4300 3800
 Wire Wire Line
-	4300 3050 4300 3400
+	4300 3050 4300 3350
+Wire Wire Line
+	4300 3350 4300 3400
 Wire Wire Line
 	3900 3300 3900 3350
@@
 Connection ~ 4300 3350
 Wire Wire Line
-	4550 2750 4500 2750
-Wire Wire Line
 	1200 5450 1200 3400
 Wire Wire Line
@@
 Connection ~ 3300 1100
 Wire Wire Line
-	2950 1100 3400 1100
-Wire Wire Line
-	1700 2550 2350 2550
+	2950 1100 3050 1100
+Wire Wire Line
+	3050 1100 3300 1100
+Wire Wire Line
+	3300 1100 3400 1100
+Wire Wire Line
+	1700 2550 2150 2550
+Wire Wire Line
+	2150 2550 2350 2550
 Wire Wire Line
 	2150 2600 2150 2550
 Connection ~ 2150 2550
 Wire Wire Line
-	3450 2750 4100 2750
+	3450 2750 3900 2750
+Wire Wire Line
+	3900 2750 4100 2750
 Text Label 3450 2750 0    60   ~ 0
 LED_VCC
@@
 L LED D2
 U 1 1 550E272C
-P 6450 4450
-F 0 "D2" V 6300 4500 50  0000 C CNN
-F 1 "LED" H 6450 4350 50  0000 C CNN
-F 2 "Pin_Headers:Pin_Header_Straight_1x02" H 6450 4450 60  0001 C CNN
-F 3 "" H 6450 4450 60  0000 C CNN
-	1    6450 4450
+P 6450 4300
+F 0 "D2" V 6300 4350 50  0000 C CNN
+F 1 "LED" H 6450 4200 50  0000 C CNN
+F 2 "Pin_Headers:Pin_Header_Straight_1x02" H 6450 4300 60  0001 C CNN
+F 3 "" H 6450 4300 60  0000 C CNN
+	1    6450 4300
 	0    1    1    0
 $EndComp
 Wire Wire Line
-	6150 4250 6150 2750
-Wire Wire Line
-	6150 2750 5050 2750
-Wire Wire Line
-	6450 4250 6450 2550
-Wire Wire Line
-	6450 2550 3300 2550
+	6150 4100 6150 2750
+Wire Wire Line
+	6150 2750 4500 2750
+Wire Wire Line
+	6450 4100 6450 2550
+Wire Wire Line
+	6450 2550 2750 2550
 Text Label 1350 5050 1    60   ~ 0
 LED_SEL_1
@@
 AMP_SEL
 Wire Wire Line
-	1400 1200 1400 1650
+	1400 1200 1400 1500
+Wire Wire Line
+	1400 1500 1400 1650
 Wire Wire Line
 	1400 1200 1300 1200
@@
 	1    0    0    -1
 $EndComp
-$Comp
-L R R13
-U 1 1 550E5632
-P 6450 5000
-F 0 "R13" H 6550 5050 40  0000 C CNN
-F 1 "10" H 6550 4950 40  0000 C CNN
-F 2 "Resistors_ThroughHole:Resistor_Horizontal_RM10mm" V 6380 5000 30  0001 C CNN
-F 3 "" H 6450 5000 30  0000 C CNN
-	1    6450 5000
-	1    0    0    -1
-$EndComp
-Wire Wire Line
-	6450 4750 6450 4650
-Wire Wire Line
-	6150 4750 6150 4650
-Wire Wire Line
-	6150 5250 6150 5400
-Wire Wire Line
-	6150 5400 6450 5400
-Wire Wire Line
-	6450 5400 6450 5250
+Wire Wire Line
+	6150 5400 6300 5400
+Wire Wire Line
+	6300 5400 6450 5400
 Wire Wire Line
 	6300 6000 6300 5400
@@
 	8200 5500 8200 5100
 Wire Wire Line
-	8050 5100 8300 5100
+	8050 5100 8200 5100
+Wire Wire Line
+	8200 5100 8300 5100
 Wire Wire Line
 	8300 4900 7500 4900
 Wire Wire Line
-	7500 4900 7500 5500
+	7500 4900 7500 5100
+Wire Wire Line
+	7500 5100 7500 5500
 Wire Wire Line
 	7500 5500 7550 5500
@@
 $EndComp
 Wire Wire Line
-	7500 4400 8300 4400
-Wire Wire Line
-	7500 4500 8150 4500
+	7500 4400 7650 4400
+Wire Wire Line
+	7650 4400 8300 4400
+Wire Wire Line
+	7500 4500 7900 4500
+Wire Wire Line
+	7900 4500 8150 4500
 Wire Wire Line
 	8150 4500 8150 4600
@@
 	4600 1600 4600 1650
 Wire Wire Line
-	4250 1100 4700 1100
-Wire Wire Line
-	4600 1050 4600 1200
+	4250 1100 4600 1100
+Wire Wire Line
+	4600 1100 4700 1100
+Wire Wire Line
+	4600 1050 4600 1100
+Wire Wire Line
+	4600 1100 4600 1200
 $Comp
 L GND #PWR026
@@
 $EndComp
 Wire Wire Line
-	9600 2350 9600 2800
+	9600 2350 9600 2450
+Wire Wire Line
+	9600 2450 9600 2550
+Wire Wire Line
+	9600 2550 9600 2650
+Wire Wire Line
+	9600 2650 9600 2750
+Wire Wire Line
+	9600 2750 9600 2800
 Wire Wire Line
 	9600 2350 9450 2350
@@
 Connection ~ 9600 2750
 Wire Wire Line
-	8900 2250 8900 2550
+	8900 2250 8900 2350
+Wire Wire Line
+	8900 2350 8900 2450
+Wire Wire Line
+	8900 2450 8900 2550
 Wire Wire Line
 	8900 2550 8950 2550
@@
 $EndComp
 Wire Wire Line
-	8750 2400 8750 2750
+	8750 2400 8750 2650
+Wire Wire Line
+	8750 2650 8750 2750
 Wire Wire Line
 	8750 2750 8950 2750
@@
 $EndComp
 $Comp
-L FUSE F?
+L FUSE F1
 U 1 1 55292D4A
 P 1700 1100
-F 0 "F?" H 1800 1150 40  0000 C CNN
+F 0 "F1" H 1800 1150 40  0000 C CNN
 F 1 "FUSE" H 1600 1050 40  0000 C CNN
-F 2 "" H 1700 1100 60  0000 C CNN
+F 2 "Capacitors_ThroughHole:Capacitor6MMDiscRM5" H 1700 1100 60  0001 C CNN
 F 3 "" H 1700 1100 60  0000 C CNN
 	1    1700 1100
@@
 Wire Wire Line
 	1450 1100 1300 1100
+Wire Wire Line
+	6150 5150 6150 5400
+Wire Wire Line
+	6450 5400 6450 5150
+Wire Wire Line
+	6150 4650 6150 4500
+Wire Wire Line
+	6450 4650 6450 4500
 $EndSCHEMATC

Commit message: sort of shaped up
Connections:
- wire segments 218 -> 184
Changed lines of the file:
@@
 	3250 6300 3250 6250
 Wire Wire Line
-	3100 5650 3250 5650
-Wire Wire Line
-	3250 5650 3400 5650
+	3100 5650 3400 5650
 Wire Wire Line
 	3250 5750 3250 5650
@@
 	3700 5950 3700 5850
 Wire Wire Line
-	3700 5100 3700 5400
-Wire Wire Line
-	3700 5400 3700 5450
+	3700 5100 3700 5450
 Wire Wire Line
 	3300 5350 3300 5400
@@
 	4400 4900 4500 4900
 Wire Wire Line
-	1950 1100 2100 1100
-Wire Wire Line
-	2100 1100 2350 1100
-Wire Wire Line
-	2350 1100 2450 1100
-Wire Wire Line
-	2100 950  2100 1100
-Wire Wire Line
-	2100 1100 2100 1200
+	1950 1100 2450 1100
+Wire Wire Line
+	2100 950  2100 1200
 Connection ~ 2100 1100
 Wire Wire Line
-	2350 1000 2350 1100
-Wire Wire Line
-	2350 1100 2350 1200
+	2350 1000 2350 1200
 Connection ~ 2350 1100
 Wire Wire Line
-	3150 4800 3300 4800
-Wire Wire Line
-	3300 4800 3500 4800
+	3150 4800 3500 4800
 Wire Wire Line
 	3300 4850 3300 4800
@@
 	3800 7200 3800 7150
 Wire Wire Line
-	3650 6550 3800 6550
-Wire Wire Line
-	3800 6550 3950 6550
+	3650 6550 3950 6550
 Wire Wire Line
 	3800 6650 3800 6550
@@
 	4250 6850 4250 6750
 Wire Wire Line
-	4250 6050 4250 6200
-Wire Wire Line
-	4250 6200 4250 6350
+	4250 6050 4250 6350
 Wire Wire Line
 	4350 6200 4250 6200
@@
 	5000 5800 4950 5800
 Wire Wire Line
-	4950 5800 4950 6200
-Wire Wire Line
-	4950 6200 4950 6600
+	4950 5800 4950 6600
 Wire Wire Line
 	4950 6600 5000 6600
@@
 Connection ~ 4950 6200
 Wire Wire Line
-	5300 6000 5300 6200
-Wire Wire Line
-	5300 6200 5300 6400
+	5300 6000 5300 6400
 Wire Wire Line
 	5400 6200 5300 6200
@@
 	2100 4050 2100 4000
 Wire Wire Line
-	1950 3400 2100 3400
-Wire Wire Line
-	2100 3400 2250 3400
+	1950 3400 2250 3400
 Wire Wire Line
 	2100 3500 2100 3400
@@
 	2550 3700 2550 3600
 Wire Wire Line
-	2550 2850 2550 3150
-Wire Wire Line
-	2550 3150 2550 3200
+	2550 2850 2550 3200
 Wire Wire Line
 	2150 3100 2150 3150
@@
 	3850 4250 3850 4200
 Wire Wire Line
-	3700 3600 3850 3600
-Wire Wire Line
-	3850 3600 4000 3600
+	3700 3600 4000 3600
 Wire Wire Line
 	3850 3700 3850 3600
@@
 	4300 3900 4300 3800
 Wire Wire Line
-	4300 3050 4300 3350
-Wire Wire Line
-	4300 3350 4300 3400
+	4300 3050 4300 3400
 Wire Wire Line
 	3900 3300 3900 3350
@@
 Connection ~ 3300 1100
 Wire Wire Line
-	2950 1100 3050 1100
-Wire Wire Line
-	3050 1100 3300 1100
-Wire Wire Line
-	3300 1100 3400 1100
-Wire Wire Line
-	1700 2550 2150 2550
-Wire Wire Line
-	2150 2550 2350 2550
+	2950 1100 3400 1100
+Wire Wire Line
+	1700 2550 2350 2550
 Wire Wire Line
 	2150 2600 2150 2550
 Connection ~ 2150 2550
 Wire Wire Line
-	3450 2750 3900 2750
-Wire Wire Line
-	3900 2750 4100 2750
+	3450 2750 4100 2750
 Text Label 3450 2750 0    60   ~ 0
 LED_VCC
@@
 AMP_SEL
 Wire Wire Line
-	1400 1200 1400 1500
-Wire Wire Line
-	1400 1500 1400 1650
+	1400 1200 1400 1650
 Wire Wire Line
 	1400 1200 1300 1200
@@
 $EndComp
 Wire Wire Line
-	6150 5400 6300 5400
-Wire Wire Line
-	6300 5400 6450 5400
+	6150 5400 6450 5400
 Wire Wire Line
 	6300 6000 6300 5400
@@
 F 3 "" H 7850 5500 60  0000 C CNN
 	1    7850 5500
-	1    0    0    -1
+	-1   0    0    -1
 $EndComp
 Wire Wire Line
@@
 	8200 5500 8200 5100
 Wire Wire Line
-	8050 5100 8200 5100
-Wire Wire Line
-	8200 5100 8300 5100
+	8050 5100 8300 5100
 Wire Wire Line
 	8300 4900 7500 4900
 Wire Wire Line
-	7500 4900 7500 5100
-Wire Wire Line
-	7500 5100 7500 5500
+	7500 4900 7500 5500
 Wire Wire Line
 	7500 5500 7550 5500
@@
 $EndComp
 Wire Wire Line
-	7500 4400 7650 4400
-Wire Wire Line
-	7650 4400 8300 4400
-Wire Wire Line
-	7500 4500 7900 4500
-Wire Wire Line
-	7900 4500 8150 4500
+	7500 4400 8300 4400
+Wire Wire Line
+	7500 4500 8150 4500
 Wire Wire Line
 	8150 4500 8150 4600
@@
 	4600 1600 4600 1650
 Wire Wire Line
-	4250 1100 4600 1100
-Wire Wire Line
-	4600 1100 4700 1100
-Wire Wire Line
-	4600 1050 4600 1100
-Wire Wire Line
-	4600 1100 4600 1200
+	4250 1100 4700 1100
+Wire Wire Line
+	4600 1050 4600 1200
 $Comp
 L GND #PWR026
@@
 $EndComp
 Wire Wire Line
-	9600 2350 9600 2450
-Wire Wire Line
-	9600 2450 9600 2550
-Wire Wire Line
-	9600 2550 9600 2650
-Wire Wire Line
-	9600 2650 9600 2750
-Wire Wire Line
-	9600 2750 9600 2800
+	9600 2350 9600 2800
 Wire Wire Line
 	9600 2350 9450 2350
@@
 Connection ~ 9600 2750
 Wire Wire Line
-	8900 2250 8900 2350
-Wire Wire Line
-	8900 2350 8900 2450
-Wire Wire Line
-	8900 2450 8900 2550
+	8900 2250 8900 2550
 Wire Wire Line
 	8900 2550 8950 2550
@@
 $EndComp
 Wire Wire Line
-	8750 2400 8750 2650
-Wire Wire Line
-	8750 2650 8750 2750
+	8750 2400 8750 2750
 Wire Wire Line
 	8750 2750 8950 2750
