File: electronics/digital/digital.sch (KiCad schematic (older format))
At the start: 58 parts, among them J1 USB_A, J2 USB_A, J3 RJ45, P1 POWER_IN, P10 AMP_POWER_OUT, P11 CONTROL, P2 3V3_IN, P3 USB_CABLE, P4 USB_CABLE, P5 NETWORK_CABLE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

Commit message: work on pcb
Parts:
- C2, C4: footprint Capacitors_ThroughHole:Capacitor6MMDiscRM5 -> SMD_Packages:SMD-1206
Changed lines of the file:
@@
 F 0 "C2" H 2350 1500 40  0000 L CNN
 F 1 "100n" H 2356 1315 40  0000 L CNN
-F 2 "Capacitors_ThroughHole:Capacitor6MMDiscRM5" H 2388 1250 30  0001 C CNN
+F 2 "SMD_Packages:SMD-1206" H 2388 1250 30  0001 C CNN
 F 3 "" H 2350 1400 60  0000 C CNN
 	1    2350 1400
@@
 F 0 "C4" H 3300 1500 40  0000 L CNN
 F 1 "100n" H 3306 1315 40  0000 L CNN
-F 2 "Capacitors_ThroughHole:Capacitor6MMDiscRM5" H 3338 1250 30  0001 C CNN
+F 2 "SMD_Packages:SMD-1206" H 3338 1250 30  0001 C CNN
 F 3 "" H 3300 1400 60  0000 C CNN
 	1    3300 1400

Commit message: placed everything
Parts:
- removed P11: CONTROL, Pin_Headers:Pin_Header_Straight_1x05, symbol CONN_01X05
- added P11: CONTROL, Pin_Headers:Pin_Header_Straight_1x04, symbol CONN_01X04
Connections:
- wire segments 184 -> 217

Commit message: fuck 3v3
Parts:
- added C10: 10u, Capacitors_ThroughHole:Capacitor10x16RM5, symbol CP2
- added C11, C9: 100n, Capacitors_ThroughHole:Capacitor6MMDiscRM5, symbol C
- added D3: TL431, Discret:TO92-123, symbol TL431
- added P12: ADC, Pin_Headers:Pin_Header_Straight_1x03, symbol CONN_01X03
- added R12, R22, R24: 10k, Resistors_ThroughHole:Resistor_Horizontal_RM10mm, symbol R
- added R13: Photores, Pin_Headers:Pin_Header_Straight_1x02, symbol Photores
- added R23: 2.2k, Resistors_ThroughHole:Resistor_Horizontal_RM10mm, symbol R
- added U2: MCP3001, Power_Integrations:SO-8, symbol MCP3001
Connections:
- wire segments 217 -> 208
Other:
- moved on the sheet: BT1, C6, C7, C8, J1, J2, P3, P4, P6, P7, P8, P9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
