File: electronics/digital/digital.sch (KiCad schematic (older format))
At the start: 69 parts, among them J1 USB_A, J2 USB_A, J3 RJ45, P1 POWER_IN, P10 AMP_POWER_OUT, P11 CONTROL, P12 ADC, P2 3V3_IN, P3 USB_CABLE, P4 USB_CABLE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

Commit message: add some GND pads
Parts:
- removed P12: ADC, Pin_Headers:Pin_Header_Straight_1x03, symbol CONN_01X03
- added P11: CONTROL, symbol CONN_01X05
- added P13: I2C 2, Pin_Headers:Pin_Header_Straight_1x02, symbol CONN_01X02
- P12: renamed from P11; value CONTROL -> ADC_SPI
- P9: value I2C -> I2C 1
Connections:
- wire segments 208 -> 212
Other:
- moved on the sheet: P9
Changed lines of the file:
@@
 L CONN_01X02 P9
 U 1 1 550E901A
-P 7600 5000
-F 0 "P9" H 7600 5150 50  0000 C CNN
-F 1 "I2C" H 7600 4850 50  0000 C CNN
-F 2 "Pin_Headers:Pin_Header_Straight_1x02" H 7600 5000 60  0001 C CNN
-F 3 "" H 7600 5000 60  0000 C CNN
-	1    7600 5000
+P 7500 5000
+F 0 "P9" H 7300 5150 50  0000 C CNN
+F 1 "I2C 1" H 7500 4850 50  0000 C CNN
+F 2 "Pin_Headers:Pin_Header_Straight_1x02" H 7500 5000 60  0001 C CNN
+F 3 "" H 7500 5000 60  0000 C CNN
+	1    7500 5000
 	-1   0    0    -1
 $EndComp
 Wire Wire Line
-	7800 4950 8600 4950
-Wire Wire Line
-	7800 5050 8450 5050
+	7700 4950 8600 4950
+Wire Wire Line
+	7700 5050 8450 5050
 Wire Wire Line
 	8450 5050 8450 5150
@@
 	8200 4200 8200 4300
 Wire Wire Line
-	7950 4800 7950 4950
+	7950 4800 7950 5300
 Connection ~ 7950 4950
 Wire Wire Line
-	8200 4800 8200 5050
+	8200 4800 8200 5400
 Connection ~ 8200 5050
 $Comp
@@
 	1000 5650 2600 5650
 $Comp
-L CONN_01X04 P11
+L CONN_01X04 P12
 U 1 1 5533A385
-P 800 5800
-F 0 "P11" H 800 6050 50  0000 C CNN
-F 1 "CONTROL" V 900 5800 50  0000 C CNN
-F 2 "Pin_Headers:Pin_Header_Straight_1x04" H 800 5800 60  0001 C CNN
-F 3 "" H 800 5800 60  0000 C CNN
-	1    800  5800
-	-1   0    0    1
+P 9450 2550
+F 0 "P12" H 9450 2800 50  0000 C CNN
+F 1 "ADC_SPI" V 9550 2550 50  0000 C CNN
+F 2 "Pin_Headers:Pin_Header_Straight_1x04" H 9450 2550 60  0001 C CNN
+F 3 "" H 9450 2550 60  0000 C CNN
+	1    9450 2550
+	1    0    0    1
 $EndComp
 $Comp
@@
 	1    0    0    -1
 $EndComp
-$Comp
-L CONN_01X03 P12
-U 1 1 55356EB4
-P 9400 2600
-F 0 "P12" H 9400 2800 50  0000 C CNN
-F 1 "ADC" V 9500 2600 50  0000 C CNN
-F 2 "Pin_Headers:Pin_Header_Straight_1x03" H 9400 2600 60  0001 C CNN
-F 3 "" H 9400 2600 60  0000 C CNN
-	1    9400 2600
-	1    0    0    1
-$EndComp
-Wire Wire Line
-	9200 2500 9150 2500
-Wire Wire Line
-	9150 2600 9200 2600
-Wire Wire Line
-	9200 2700 9150 2700
+Wire Wire Line
+	9250 2500 9150 2500
+Wire Wire Line
+	9150 2600 9250 2600
+Wire Wire Line
+	9250 2700 9150 2700
 $Comp
 L GND #PWR049
@@
 Wire Wire Line
 	7750 1800 7750 1850
+$Comp
+L GND #PWR060
+U 1 1 553FDB51
+P 9200 2400
+F 0 "#PWR060" H 9200 2150 60  0001 C CNN
+F 1 "GND" H 9200 2250 60  0001 C CNN
+F 2 "" H 9200 2400 60  0000 C CNN
+F 3 "" H 9200 2400 60  0000 C CNN
+	1    9200 2400
+	0    1    1    0
+$EndComp
+Wire Wire Line
+	9200 2400 9250 2400
+$Comp
+L CONN_01X05 P11
+U 1 1 553FE851
+P 800 5750
+F 0 "P11" H 800 6050 50  0000 C CNN
+F 1 "CONTROL" V 900 5750 50  0000 C CNN
+F 2 "" H 800 5750 60  0000 C CNN
+F 3 "" H 800 5750 60  0000 C CNN
+	1    800  5750
+	-1   0    0    1
+$EndComp
+$Comp
+L GND #PWR061
+U 1 1 553FF2F4
+P 1050 5550
+F 0 "#PWR061" H 1050 5300 60  0001 C CNN
+F 1 "GND" H 1050 5400 60  0001 C CNN
+F 2 "" H 1050 5550 60  0000 C CNN
+F 3 "" H 1050 5550 60  0000 C CNN
+	1    1050 5550
+	0    -1   -1   0
+$EndComp
+Wire Wire Line
+	1050 5550 1000 5550
+$Comp
+L CONN_01X02 P13
+U 1 1 55400B41
+P 7500 5350
+F 0 "P13" H 7300 5500 50  0000 C CNN
+F 1 "I2C 2" H 7500 5200 50  0000 C CNN
+F 2 "Pin_Headers:Pin_Header_Straight_1x02" H 7500 5350 60  0001 C CNN
+F 3 "" H 7500 5350 60  0000 C CNN
+	1    7500 5350
+	-1   0    0    -1
+$EndComp
+Wire Wire Line
+	7950 5300 7700 5300
+Wire Wire Line
+	8200 5400 7700 5400
 $EndSCHEMATC

Commit message: fix values of referance voltage regulator
Parts:
- R22: value 10k -> 560
- R23: value 2.2k -> 0
- R24: value 10k -> DNP
Changed lines of the file:
@@
 P 7050 2950
 F 0 "R22" H 7150 3000 40  0000 C CNN
-F 1 "10k" H 7150 2900 40  0000 C CNN
+F 1 "560" H 7150 2900 40  0000 C CNN
 F 2 "Resistors_ThroughHole:Resistor_Horizontal_RM10mm" V 6980 2950 30  0001 C CNN
 F 3 "" H 7050 2950 30  0000 C CNN
@@
 P 7050 4250
 F 0 "R24" H 7150 4300 40  0000 C CNN
-F 1 "10k" H 7150 4200 40  0000 C CNN
+F 1 "DNP" H 7150 4200 40  0000 C CNN
 F 2 "Resistors_ThroughHole:Resistor_Horizontal_RM10mm" V 6980 4250 30  0001 C CNN
 F 3 "" H 7050 4250 30  0000 C CNN
@@
 P 7050 3550
 F 0 "R23" H 7150 3600 40  0000 C CNN
-F 1 "2.2k" H 7150 3500 40  0000 C CNN
+F 1 "0" H 7150 3500 40  0000 C CNN
 F 2 "Resistors_ThroughHole:Resistor_Horizontal_RM10mm" V 6980 3550 30  0001 C CNN
 F 3 "" H 7050 3550 30  0000 C CNN
