File: electronics/digital/digital.kicad_pcb (KiCad board)
At the start: 2 copper layers, 75 parts, among them J1 USB_A, J2 USB_A, J3 RJ45, P1 POWER_IN, P10 AMP_POWER_OUT, P11 CONTROL, P12 ADC, P2 3V3_IN, P3 USB_CABLE, P4 USB_CABLE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

Commit message: add some GND pads
Parts:
- added P13: I2C 2, Pin_Headers:Pin_Header_Straight_1x02, F.Cu at (224.8, 106.7)
- P11: footprint Pin_Headers:Pin_Header_Straight_1x04 -> Pin_Headers:Pin_Header_Straight_1x05
- P12: value ADC -> ADC_SPI; footprint Pin_Headers:Pin_Header_Straight_1x03 -> Pin_Headers:Pin_Header_Straight_1x04
- P9: value I2C -> I2C 1
- moved R1 2.54 mm to (217.8, 99.1)
- moved R15 2.54 mm to (217.8, 102.9)
- moved P12 1.27 mm to (216.5, 135.9)
- moved P11 1.27 mm to (228.0, 97.8)
Connections:
- J3 pad Hole: GND -> (no net)
Routing:
- net GND: track 211.9 -> 218.8 mm
- net /LED_PWM: track 38.0 -> 35.5 mm
- net /LED_SEL_1: track 21.7 -> 19.2 mm
- net /LED_SEL_2: track 10.8 -> 8.30 mm
- net Net-(Q8-PadD): track 35.6 -> 33.1 mm
- net Net-(Q6-Pad2): track 20.5 -> 22.9 mm
- net Net-(D2-Pad2): track 6.98 -> 8.78 mm
- net /SDA: track 16.9 -> 18.1 mm
- net /AMP_SEL: track 6.13 -> 6.88 mm

Commit message: work on adc
Parts:
- R22: value 10k -> 560
- R23: value 2.2k -> 0
- R24: value 10k -> DNP
Changed lines of the file:
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@@
-(kicad_pcb (version 4) (host pcbnew "(after 2015-jan-16 BZR unknown)-product")
+(kicad_pcb (version 4) (host pcbnew "(after 2015-may-01 BZR unknown)-product")
   (general
     (links 164)
     (no_connects 5)
-    (area 186.69 48.732 264.870001 153.035001)
+    (area 0 0 0 0)
     (thickness 1.6)
     (drawings 1)
@@
     (visible_elements FFFEFF7F)
     (pcbplotparams
-      (layerselection 0x00000_80000000)
+      (layerselection 0x00030_80000001)
       (usegerberextensions false)
       (excludeedgelayer true)
@@
       (outputformat 5)
       (mirror false)
-      (drillshape 1)
+      (drillshape 0)
       (scaleselection 1)
       (outputdirectory ../prints/))
@@
       (effects (font (size 1 1) (thickness 0.15)))
     )
-    (fp_text value 10k (at 3.81 3.81 180) (layer F.SilkS) hide
+    (fp_text value 560 (at 3.81 3.81 180) (layer F.SilkS) hide
       (effects (font (size 1 1) (thickness 0.15)))
     )
@@
       (effects (font (size 1 1) (thickness 0.15)))
     )
-    (fp_text value 2.2k (at 3.81 3.81 180) (layer F.SilkS) hide
+    (fp_text value 0 (at 3.81 3.81 180) (layer F.SilkS) hide
       (effects (font (size 1 1) (thickness 0.15)))
     )
@@
       (effects (font (size 1 1) (thickness 0.15)))
     )
-    (fp_text value 10k (at 3.81 3.81) (layer F.SilkS) hide
+    (fp_text value DNP (at 3.81 3.81) (layer F.SilkS) hide
       (effects (font (size 1 1) (thickness 0.15)))
     )
@@
   (segment (start 246.38 123.825) (end 254 123.825) (width 0.8) (layer B.Cu) (net 33))
   (segment (start 245.745 123.19) (end 246.38 123.825) (width 0.8) (layer B.Cu) (net 33))
-  (segment (start 224.79 107.95) (end 220.98 107.95) (width 0.8) (layer B.Cu) (net 34) (status 400000))
-  (segment (start 220.345 108.585) (end 220.345 110.871) (width 0.8) (layer B.Cu) (net 34) (status 800000))
+  (segment (start 224.79 107.95) (end 220.98 107.95) (width 0.8) (layer B.Cu) (net 34))
+  (segment (start 220.345 108.585) (end 220.345 110.871) (width 0.8) (layer B.Cu) (net 34))
   (segment (start 220.98 107.95) (end 220.345 108.585) (width 0.8) (layer B.Cu) (net 34))
-  (segment (start 227.965 107.95) (end 224.79 107.95) (width 0.8) (layer B.Cu) (net 34) (status C00000))
+  (segment (start 227.965 107.95) (end 224.79 107.95) (width 0.8) (layer B.Cu) (net 34))
   (segment (start 231.775 107.95) (end 227.965 107.95) (width 0.8) (layer B.Cu) (net 34))
-  (segment (start 224.79 105.41) (end 219.71 105.41) (width 0.8) (layer B.Cu) (net 35) (status 400000))
-  (segment (start 219.075 106.045) (end 219.075 110.871) (width 0.8) (layer B.Cu) (net 35) (status 800000))
+  (segment (start 224.79 105.41) (end 219.71 105.41) (width 0.8) (layer B.Cu) (net 35))
+  (segment (start 219.075 106.045) (end 219.075 110.871) (width 0.8) (layer B.Cu) (net 35))
   (segment (start 219.71 105.41) (end 219.075 106.045) (width 0.8) (layer B.Cu) (net 35))
-  (segment (start 227.965 105.41) (end 224.79 105.41) (width 0.8) (layer B.Cu) (net 35) (status C00000))
+  (segment (start 227.965 105.41) (end 224.79 105.41) (width 0.8) (layer B.Cu) (net 35))
   (segment (start 229.87 105.41) (end 227.965 105.41) (width 0.8) (layer B.Cu) (net 35))
   (segment (start 231.775 104.775) (end 230.505 104.775) (width 0.8) (layer B.Cu) (net 35))
